File: Design-Files/DuressBadge-v1.1/DuressBadge.brd (EAGLE design)
At the start: 55 x 40 mm, 52 parts, among them SW1 GX10700, SW2 GX10700, Y1 RESONATORSMD

Commit message: Change: folder structure
Parts:
- removed LED_D9_DNP: LED3MM, LowPowerLab:LED3MM
- removed USB_TOP: USB_5PINSLOTS_HOLES, LowPowerLab:USB-B-MICRO_5PADS_SLOTS_HOLES
- added J1: 12401832E402A, Connector_USB:12401832E402A
- moved R12 48.4 mm to (18.7, 2.40)
- moved C4 42.9 mm to (17.9, 6.17), flipped to the bottom, turned to 90 degrees
- moved C2 41.4 mm to (51.9, 17.9)
- moved LIS3DH 39.8 mm to (23.4, 2.89)
- moved C8 38.3 mm to (52.1, 13.1), turned to 90 degrees
- moved R6 37.5 mm to (50.5, 17.9)
- moved R5 37.1 mm to (48.9, 17.9)
- moved C1 36.7 mm to (75.2, 24.7)
- moved C3 35.9 mm to (73.0, 24.9)
- moved R9 35.2 mm to (43.9, 2.31), turned to 90 degrees
- moved R10 34.2 mm to (42.3, 2.31), turned to 90 degrees
- moved U$31 32.7 mm to (0.56, 5.10)
- moved TAG-ICSP 29.9 mm to (27.6, 9.99)
- moved C14 28.8 mm to (50.6, 13.1), turned to 90 degrees
- moved TP1 28.4 mm to (35.8, 7.26)
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Connections:
- removed net DTR1: C3.1, USB_TOP.D-
- net D0_RX: now also J1.B6; no longer USB_TOP.D+
- net D1_TX: now also J1.B7; no longer USB_TOP.ID
- net GND: now also J1.A1, J1.A12, J1.B1, J1.B12; no longer LED_D9_DNP.MINUS, USB_TOP.GND, USB_TOP.MT5, USB_TOP.MT6, USB_TOP.MT7, USB_TOP.MT8, USB_TOP.P$1, USB_TOP.P$3, USB_TOP.P$4, USB_TOP.P$5, USB_TOP.P$6, USB_TOP.P$7
- net N$6: no longer LED_D9_DNP.PLUS
- net VUSB: now also J1.A4, J1.A9, J1.B4, J1.B9; no longer USB_TOP.VBUS
Routing:
- net VCC: track 133.8 -> 1641.6 mm, vias 1 -> 7
- net VBAT: track 124.1 -> 497.9 mm, vias 5 -> 7
- net RST: track 44.1 -> 252.4 mm, vias 5 -> 2
- net D3: track 41.5 -> 189.5 mm
- net N$2: track 71.6 -> 206.3 mm, vias 4 -> 2
- net VUSB: track 28.8 -> 144.2 mm
- net A4_SDA: track 22.8 -> 114.6 mm, vias 2 -> 1
- net A7_VMON: track 33.3 -> 102.3 mm, vias 2 -> 1
- net A5_SCL: track 18.7 -> 87.6 mm
- net A2_CHGSTAT: track 21.7 -> 90.1 mm, vias 2 -> 4
- net D11_MOSI: track 25.2 -> 80.6 mm
- net D13_SCK: track 15.1 -> 67.7 mm
- net ANT: track 7.31 -> 56.2 mm
- net A3_RGB_DATA: track 16.9 -> 63.2 mm, vias 2 -> 1
- net D4_RGBPWR: track 9.94 -> 50.7 mm
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Other:
- board size 55 x 40 mm -> 70.2 x 22.6 mm

Commit message: Add files via upload
Parts:
- added U$2: W25Q40CLSNIG, W25Q40CLSNIG:USON
Connections:
- net GND: now also U$2.4
- net VCC: now also U$2.8, U$2.GND1
Routing:
- net VCC: track 1641.6 -> 764.8 mm
Changed lines of the file:
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@@
 <attribute name="VOLTAGE_RATING" value="NA" x="66.802" y="30.353" size="1.778" layer="27" display="off"/>
 </element>
+<element name="U$2" library="W25Q40CLSNIG" package="USON" value="W25Q40CLSNIG" x="8.255" y="1.524" smashed="yes"/>
 </elements>
 <signals>
@@
 <contactref element="J1" pad="B12"/>
 <contactref element="J1" pad="B1"/>
+<contactref element="U$2" pad="4"/>
 <wire x1="69.302" y1="33.653" x2="69.552" y2="35.353" width="0" layer="19" extent="1-1"/>
 <wire x1="64.052" y1="35.353" x2="69.552" y2="35.353" width="0" layer="19" extent="1-1"/>
@@
 <wire x1="10.3378" y1="39.2176" x2="10.3378" y2="39.1668" width="0" layer="19" extent="1-16"/>
 <wire x1="75.184" y1="23.8896" x2="69.302" y2="33.653" width="0" layer="19" extent="1-1"/>
+<wire x1="7.105" y1="0.774" x2="13.414" y2="5.776" width="0" layer="19" extent="1-1"/>
 </signal>
 <signal name="D10_SS">
@@
 <wire x1="56.8462" y1="33.8582" x2="24.8746" y2="1.8866" width="0.254" layer="1"/>
 <wire x1="46.736" y1="30.1498" x2="44.9078" y2="28.3216" width="0.254" layer="1"/>
-<wire x1="-431.289428125" y1="20.3962" x2="-425.0162125" y2="14.122984375" width="0.254" layer="16"/>
-<wire x1="23.5492" y1="4.0104" x2="-425.0162125" y2="14.122984375" width="0.254" layer="16"/>
+<wire x1="23.5492" y1="4.0104" x2="36.321771875" y2="4.0104" width="0.254" layer="16"/>
+<wire x1="56.263571875" y1="23.9522" x2="36.321771875" y2="4.0104" width="0.254" layer="16"/>
 <wire x1="48.1234" y1="25.106" x2="48.1234" y2="9.0548" width="0.381" layer="1"/>
 <wire x1="44.6792" y1="28.0918" x2="45.1358" y2="27.6352" width="0.381" layer="1"/>
 <wire x1="44.6792" y1="28.0918" x2="44.9078" y2="28.3216" width="0.254" layer="1"/>
-<wire x1="-431.289428125" y1="20.3962" x2="37.620515625" y2="20.3962" width="0.381" layer="1"/>
-<wire x1="37.620515625" y1="20.3962" x2="45.3898" y2="1.4614" width="0.381" layer="1"/>
+<wire x1="56.263571875" y1="23.9522" x2="41.954859375" y2="9.832815625" width="0.381" layer="1"/>
+<wire x1="41.954859375" y1="9.832815625" x2="45.3898" y2="1.4614" width="0.381" layer="1"/>
 <wire x1="28.379553125" y1="11.077278125" x2="38.729475" y2="21.4272" width="0.381" layer="16"/>
 <wire x1="28.379553125" y1="11.077278125" x2="25.4358" y2="4.2554" width="0.381" layer="16"/>
@@
 <wire x1="48.1234" y1="25.106" x2="48.1234" y2="10.6548" width="0.254" layer="1"/>
 <via x="64.8114" y="8.9762" extent="1-16" drill="0.35"/>
-<via x="-431.289428125" y="20.3962" extent="1-16" drill="0.35"/>
+<via x="56.263571875" y="23.9522" extent="1-16" drill="0.35"/>
 <via x="38.729475" y="21.4272" extent="1-16" drill="0.35"/>
 <via x="39.5382" y="20.896" extent="1-16" drill="0.35"/>
@@
 <via x="64.611" y="8.9762" extent="1-16" drill="0.35"/>
 <via x="16.4882" y="11.1504" extent="1-16" drill="0.35"/>
+<contactref element="U$2" pad="8"/>
+<contactref element="U$2" pad="GND1"/>
 <wire x1="43.8508" y1="3.1614" x2="48.1234" y2="9.0548" width="0" layer="19" extent="1-1"/>
 <wire x1="19.5158" y1="5.9434" x2="17.8562" y2="7.0222" width="0" layer="19" extent="16-16"/>
@@
 <wire x1="21.8834" y1="-7.0104" x2="21.8834" y2="-7.0104" width="0" layer="19" extent="1-16"/>
 <wire x1="26.289" y1="10.6299" x2="26.1366" y2="8.3058" width="0" layer="19" extent="16-16"/>
+<wire x1="9.405" y1="2.274" x2="21.8834" y2="-7.0104" width="0" layer="19" extent="1-1"/>
+<wire x1="8.255" y1="1.524" x2="9.405" y2="2.274" width="0" layer="19" extent="1-1"/>
 </signal>
 <signal name="D1_TX">
