File: Design-Files/DuressBadge-v1.1/DuressBadge.sch (EAGLE design)
At the start: 51 parts, among them SW1 GX10700, SW2 GX10700, Y1 RESONATORSMD

Commit message: Change: folder structure
Parts:
- removed LED_D9_DNP: LED3MM, LowPowerLab:LED3MM
- removed USB_TOP: USB_5PINSLOTS_HOLES, LowPowerLab:USB_5PINSLOTS_HOLES
- added J1: 12401832E402A, Connector_USB:12401832E402A
Connections:
- removed net DTR1: C3.1, USB_TOP.D-
- net D0_RX: now also J1.D+2; no longer USB_TOP.D+
- net D1_TX: now also J1.D-2; no longer USB_TOP.ID
- net GND: now also J1.GND1, J1.GND2, J1.GND3, J1.GND4; no longer LED_D9_DNP.MINUS, USB_TOP.GND
- net N$6: no longer LED_D9_DNP.PLUS
- net VUSB: now also J1.VBUS1, J1.VBUS2, J1.VBUS3, J1.VBUS4; no longer USB_TOP.VBUS
Other:
- moved on the sheet: C1, C13, C3, C7, JST, LDO, MCP73831, PFET, R7, R8, RCHRG, RGB_LED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

Commit message: Add files via upload
Parts:
- added U$2: W25Q40CLSNIG, W25Q40CLSNIG:W25Q40CLSNIG
Connections:
- net GND: now also U$2.GND\
- net VCC: now also U$2.VCC
