File: Design-Files/Duress_Badge_V2.0/Duress_Badge_V2.0.brd (EAGLE design)
At the start: 52 x 20 mm, 31 parts, among them SW1 GX10700

Commit message: #1 Some changes in routing
Parts:
- moved LIS3DH 0.08 mm to (26.6, 16.5)
Routing:
- net GND: track 10.8 -> 9.07 mm, vias 4 -> 5
- net VCC: track 35.0 -> 36.7 mm
- net VBAT: track 21.6 -> 22.1 mm

Commit message: #1 Pads added and Deliverables generated
Parts:
- removed U2: (no value), Seeeduino-XIAO-footprint-eagle:MOUDLE14P-2.54-21X17.8MM
- added U1: (no value), Seeeduino-XIAO-footprint-eagle:MOUDLE14P-2.54-21X17.8MM
- moved LIS3DH 0.05 mm to (26.6, 16.4)
Connections:
- net A3_RGB_DATA: now also U1.4; no longer U2.4
- net A4_SDA: now also U1.5; no longer U2.5
- net A5_SCL: now also U1.6; no longer U2.6
- net A7_VMON: now also U1.2; no longer U2.2
- net D3: now also U1.11; no longer U2.11
- net D4_RGBPWR: now also U1.3; no longer U2.3
- net D8_IR: now also U1.9; no longer U2.9
- net D9_IR: now also U1.8; no longer U2.8
- net GND: now also U1.13, U1.MP2; no longer U2.13
- net VBAT: now also U1.MP1
- net VCC: now also U1.12; no longer U2.12
Routing:
- net VBAT: track 22.1 -> 36.8 mm, vias 5 -> 7
- net GND: track 9.07 -> 13.0 mm, vias 5 -> 7
- net A5_SCL: track 25.5 -> 27.7 mm
- net D4_RGBPWR: track 48.4 -> 50.4 mm
- net VCC: track 36.7 -> 35.5 mm
Other:
- board text added: "D4"
- board text added: "GND"
- board text added: "RGB_LED"
- board text added: "VBAT"
