File: Design-Files/Duress_Badge_V2.0/Duress_Badge_V2.0.sch (EAGLE design)
At the start: 25 parts, among them SW2 GX10700, U1 113991054

Commit message: #1 Some changes in routing
Parts:
- removed C1: 0u1, LowPowerLab:CAP0603-CAP
- removed C3: 1u, LowPowerLab:CAP0603-CAP
- removed JST: M40-4010246, M40-4010246:M40-4010246
- removed SW2: GX10700, snaptron_Alan:GX10700
- removed TP1, TP2: PAD_OR_PIN_1TP, LowPowerLab:PAD_OR_PIN_1TP
- removed U$2: W25Q40CLSNIG, W25Q40CLSNIG:W25Q40CLSNIG
- removed U1: 113991054, 113991054:113991054
- added ACCEL, GND: TPB2,54, testpad:TPB2,54
- added C5: 0u1, LowPowerLab:CAP0603-CAP
- added D2, D4: TSAL4400, TSAL4400:TSAL4400
- added JST1: M40-4010246, M40-4010246:M40-4010246
- added N-FET1: N-CH, LowPowerLab:MOSFET-NCHANNEL
- added R1: 1K, LowPowerLab:RESISTOR0603-RES
- added R10, R2, R3, R9: 10k, LowPowerLab:RESISTOR0603-RES
- added SW1: GX10700, snaptron_Alan:GX10700
- added U2: (no value), Seeeduino-XIAO-footprint-eagle:MOUDLE-SEEEDUINO-XIAO
Connections:
- removed net N$1: D1.A, D3.A
- removed net RST: C1.2, C3.2, SW2.P
- removed net V_USB: U1.VUSB
- new net D3: C5.2, R3.2, SW1.P, U2.PA6_A10_D10_MOSI
- new net D8_IR: R4.2, U2.PA7_A8_D8_SCK
- new net N$3: N-FET1.G, R1.1, R2.2
- new net N$4: D2.C, D4.C, N-FET1.D
- net A3_RGB_DATA: now also U2.PA11_A3_D3; no longer U1.D3
- net A4_SDA: now also R9.1, U2.PA8_A4_D4_SDA; no longer U1.D5
- net A5_SCL: now also R10.1, U2.PA9_A5_D5_SCL; no longer U1.D4
- net A7_VMON: now also U2.PA4_A1_D1
- net D4_RGBPWR: now also U2.PA10_A2_D2; no longer U1.D2
- net D7_ACCEL: now also ACCEL.TP; no longer TP1.P$1
- net D9_IR: now also R1.2, U2.PB09_A7_D7_RX; no longer R4.2
- net GND: now also C5.1, GND.TP, JST1.1, N-FET1.S, R2.1, R3.1, U2.GND; no longer C1.1, JST.1, SW2.S, TP2.P$1, U$2.GND\, U1.GND
- net VBAT: now also D1.A, D2.A, D3.A, D4.A, JST1.2
- net VCC: now also R10.2, R9.2, SW1.S, U2.3V3; no longer JST.2, U$2.VCC, U1.VCC_3V3
Other:
- note added: "ACCELEROMETER"
- note added: "Addressable LED"
- note added: "ESP32C6"
- note removed: "ACCEL"
- moved on the sheet: C2, D1, D3, LIS3DH, N-FET, R12, R17, R5, R6

Commit message: #1 Pads added and Deliverables generated
Parts:
- renumbered U2 to U1
Connections:
- net GND: now also U1.MP2
- net VBAT: now also U1.MP1
Changed lines of the file:
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@@
 <part name="D2" library="TSAL4400" deviceset="TSAL4400" device=""/>
 <part name="D4" library="TSAL4400" deviceset="TSAL4400" device=""/>
-<part name="U2" library="Seeeduino-XIAO-footprint-eagle" deviceset="MOUDLE-SEEEDUINO-XIAO" device=""/>
 <part name="TL_FIDUCIAL" library="LowPowerLab" deviceset="FIDUCIAL" device="1.5MM"/>
 <part name="BR_FIDUCIAL" library="LowPowerLab" deviceset="FIDUCIAL" device="1.5MM"/>
@@
 <part name="R10" library="LowPowerLab" deviceset="RESISTOR" device="0603-RES" value="10k"/>
 <part name="SUPPLY4" library="SparkFun" deviceset="VCC" device="" value="3.3V"/>
+<part name="SUPPLY5" library="supply2" library_urn="urn:adsk.eagle:library:372" deviceset="GND" device=""/>
+<part name="U1" library="Seeeduino-XIAO-footprint-eagle" deviceset="MOUDLE-SEEEDUINO-XIAO" device=""/>
 </parts>
 <sheets>
@@
 <attribute name="VALUE" x="173.228" y="-87.884" size="1.27" layer="96" rot="R270"/>
 </instance>
-<instance part="U2" gate="G$1" x="-2.54" y="-26.67" smashed="yes">
-<attribute name="NAME" x="-24.13" y="-11.43" size="1.27" layer="95" ratio="12"/>
-<attribute name="VALUE" x="-24.13" y="-12.7" size="1.27" layer="96" ratio="12"/>
-</instance>
 <instance part="TL_FIDUCIAL" gate="G$1" x="113.03" y="-153.67" smashed="yes"/>
 <instance part="BR_FIDUCIAL" gate="G$1" x="123.19" y="-153.67" smashed="yes"/>
@@
 <attribute name="VALUE" x="54.356" y="-68.834" size="1.778" layer="96" rot="R270"/>
 </instance>
+<instance part="SUPPLY5" gate="GND" x="27.94" y="-41.91" smashed="yes" rot="R90">
+<attribute name="VALUE" x="29.845" y="-42.545" size="1.778" layer="96"/>
+</instance>
+<instance part="U1" gate="G$1" x="-2.54" y="-26.67" smashed="yes">
+<attribute name="NAME" x="-24.13" y="-11.43" size="1.27" layer="95" ratio="12"/>
+<attribute name="VALUE" x="-24.13" y="-12.7" size="1.27" layer="96" ratio="12"/>
+</instance>
 </instances>
 <busses>
 </busses>
 <nets>
-<net name="GND" class="1">
+<net name="GND" class="0">
 <segment>
 <pinref part="LIS3DH" gate="G$1" pin="GND@1"/>
@@
 <pinref part="SUPPLY2" gate="GND" pin="GND"/>
 <wire x1="25.4" y1="-19.05" x2="21.59" y2="-19.05" width="0.1524" layer="91"/>
-<pinref part="U2" gate="G$1" pin="GND"/>
+<pinref part="U1" gate="G$1" pin="GND"/>
 </segment>
 <segment>
@@
 <junction x="165.1" y="-109.22"/>
 </segment>
+<segment>
+<pinref part="SUPPLY5" gate="GND" pin="GND"/>
+<wire x1="25.4" y1="-41.91" x2="21.59" y2="-41.91" width="0.1524" layer="91"/>
+<pinref part="U1" gate="G$1" pin="MP2"/>
+</segment>
 </net>
 <net name="VCC" class="0">
@@
 <pinref part="SUPPLY3" gate="1" pin="VCC"/>
 <wire x1="21.59" y1="-22.86" x2="26.67" y2="-22.86" width="0.1524" layer="91"/>
-<pinref part="U2" gate="G$1" pin="3V3"/>
+<pinref part="U1" gate="G$1" pin="3V3"/>
 </segment>
 <segment>
@@
 <label x="-48.26" y="-30.48" size="1.778" layer="95"/>
 <label x="-48.26" y="-30.48" size="1.778" layer="95"/>
-<pinref part="U2" gate="G$1" pin="PA8_A4_D4_SDA"/>
+<pinref part="U1" gate="G$1" pin="PA8_A4_D4_SDA"/>
 </segment>
 <segment>
@@
 <wire x1="-27.94" y1="-34.29" x2="-48.26" y2="-34.29" width="0.1524" layer="91"/>
 <label x="-48.26" y="-34.29" size="1.778" layer="95"/>
-<pinref part="U2" gate="G$1" pin="PA9_A5_D5_SCL"/>
+<pinref part="U1" gate="G$1" pin="PA9_A5_D5_SCL"/>
 </segment>
 <segment>
@@
 <wire x1="-27.94" y1="-19.05" x2="-48.26" y2="-19.05" width="0.1524" layer="91"/>
 <label x="-48.26" y="-19.05" size="1.778" layer="95"/>
-<pinref part="U2" gate="G$1" pin="PA4_A1_D1"/>
+<pinref part="U1" gate="G$1" pin="PA4_A1_D1"/>
 </segment>
 </net>
@@
 <label x="176.53" y="-78.74" size="1.778" layer="95" xref="yes"/>
 <wire x1="176.53" y1="-83.82" x2="176.53" y2="-78.74" width="0.1524" layer="91"/>
+</segment>
+<segment>
+<wire x1="-41.91" y1="-41.91" x2="-27.94" y2="-41.91" width="0.1524" layer="91"/>
+<label x="-41.91" y="-41.91" size="1.27" layer="95" rot="R180" xref="yes"/>
+<pinref part="U1" gate="G$1" pin="MP1"/>
 </segment>
 </net>
@@
 <wire x1="-27.94" y1="-22.86" x2="-48.26" y2="-22.86" width="0.1524" layer="91"/>
 <label x="-48.26" y="-22.86" size="1.778" layer="95"/>
-<pinref part="U2" gate="G$1" pin="PA10_A2_D2"/>
+<pinref part="U1" gate="G$1" pin="PA10_A2_D2"/>
 </segment>
 </net>
@@
 <wire x1="-27.94" y1="-26.67" x2="-48.26" y2="-26.67" width="0.1524" layer="91"/>
 <label x="-48.26" y="-26.67" size="1.778" layer="95"/>
-<pinref part="U2" gate="G$1" pin="PA11_A3_D3"/>
+<pinref part="U1" gate="G$1" pin="PA11_A3_D3"/>
 </segment>
 </net>
@@
 <wire x1="38.1" y1="-34.29" x2="21.59" y2="-34.29" width="0.1524" layer="91"/>
 <label x="29.21" y="-34.29" size="1.778" layer="95"/>
-<pinref part="U2" gate="G$1" pin="PA7_A8_D8_SCK"/>
+<pinref part="U1" gate="G$1" pin="PA7_A8_D8_SCK"/>
 </segment>
 </net>
@@
 <label x="49.53" y="-19.05" size="1.27" layer="95" xref="yes"/>
 <wire x1="49.53" y1="-26.67" x2="49.53" y2="-27.94" width="0.1524" layer="91"/>
-<pinref part="U2" gate="G$1" pin="PA6_A10_D10_MOSI"/>
 <wire x1="49.53" y1="-26.67" x2="21.59" y2="-26.67" width="0.1524" layer="91"/>
+<pinref part="U1" gate="G$1" pin="PA6_A10_D10_MOSI"/>
 </segment>
 </net>
@@
 <wire x1="38.1" y1="-38.1" x2="21.59" y2="-38.1" width="0.1524" layer="91"/>
 <label x="29.21" y="-38.1" size="1.778" layer="95"/>
-<pinref part="U2" gate="G$1" pin="PB09_A7_D7_RX"/>
-</segment>
-</net>
+<pinref part="U1" gate="G$1" pin="PB09_A7_D7_RX"/>
+</segment>
+</net>
